File: AT89S52_dev_board.kicad_sch (KiCad schematic)
At the start: 26 parts, among them IC1 AT89S52-24PU, J1 Conn_01x20, J2 Conn_01x20, J3 Conn_01x20, J4 Conn_01x20, J5 Conn_01x20, J6 Conn_01x20, J7 Conn_02x05_Odd_Even, J8 USB_B, SW1 SW_Push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

Commit message: Assigned component values
Parts:
- C1, C3, C5, C6: value C -> 0.1u
- C10, C9: value C -> 0.47u
- C2, C4, C7, C8: value C -> 20p
- R1, R2: value R -> 4.7K
- Y1, Y2: value Crystal -> 12Mz
Changed lines of the file:
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@@
       (effects (font (size 1.27 1.27)) (justify left))
     )
-    (property "Value" "C" (id 1) (at 214.63 54.6099 0)
+    (property "Value" "0.1u" (id 1) (at 214.63 54.6099 0)
       (effects (font (size 1.27 1.27)) (justify left))
     )
@@
       (effects (font (size 1.27 1.27)) (justify left))
     )
-    (property "Value" "C" (id 1) (at 187.96 54.6099 0)
+    (property "Value" "0.1u" (id 1) (at 187.96 54.6099 0)
       (effects (font (size 1.27 1.27)) (justify left))
     )
@@
     (in_bom yes) (on_board yes) (fields_autoplaced)
     (property "Reference" "R1" (id 0) (at 232.41 142.24 90))
-    (property "Value" "R" (id 1) (at 232.41 144.78 90))
+    (property "Value" "4.7K" (id 1) (at 232.41 144.78 90))
     (property "Footprint" "Resistor_SMD:R_0805_2012Metric" (id 2) (at 232.41 150.368 90)
       (effects (font (size 1.27 1.27)) hide)
@@
     (in_bom yes) (on_board yes) (fields_autoplaced)
     (property "Reference" "R2" (id 0) (at 238.76 49.53 90))
-    (property "Value" "R" (id 1) (at 238.76 52.07 90))
+    (property "Value" "4.7K" (id 1) (at 238.76 52.07 90))
     (property "Footprint" "Resistor_SMD:R_0805_2012Metric" (id 2) (at 238.76 57.658 90)
       (effects (font (size 1.27 1.27)) hide)
@@
       (effects (font (size 1.27 1.27)) (justify left))
     )
-    (property "Value" "C" (id 1) (at 85.09 87.6299 0)
+    (property "Value" "0.47u" (id 1) (at 85.09 87.6299 0)
       (effects (font (size 1.27 1.27)) (justify left))
     )
@@
     (in_bom yes) (on_board yes) (fields_autoplaced)
     (property "Reference" "Y1" (id 0) (at 189.23 132.08 0))
-    (property "Value" "Crystal" (id 1) (at 189.23 134.62 0))
+    (property "Value" "12Mz" (id 1) (at 189.23 134.62 0))
     (property "Footprint" "Crystal:Crystal_HC49-U_Vertical" (id 2) (at 189.23 139.7 0)
       (effects (font (size 1.27 1.27)) hide)
@@
     (in_bom yes) (on_board yes) (fields_autoplaced)
     (property "Reference" "C7" (id 0) (at 63.5 86.36 90))
-    (property "Value" "C" (id 1) (at 63.5 88.9 90))
+    (property "Value" "20p" (id 1) (at 63.5 88.9 90))
     (property "Footprint" "Capacitor_SMD:C_0805_2012Metric" (id 2) (at 67.31 93.0148 0)
       (effects (font (size 1.27 1.27)) hide)
@@
       (effects (font (size 1.27 1.27)) (justify left))
     )
-    (property "Value" "C" (id 1) (at 205.74 54.6099 0)
+    (property "Value" "0.1u" (id 1) (at 205.74 54.6099 0)
       (effects (font (size 1.27 1.27)) (justify left))
     )
@@
     (in_bom yes) (on_board yes) (fields_autoplaced)
     (property "Reference" "Y2" (id 0) (at 68.58 80.01 0))
-    (property "Value" "Crystal" (id 1) (at 68.58 82.55 0))
+    (property "Value" "12Mz" (id 1) (at 68.58 82.55 0))
     (property "Footprint" "Crystal:Crystal_HC49-U_Vertical" (id 2) (at 68.58 87.63 0)
       (effects (font (size 1.27 1.27)) hide)
@@
       (effects (font (size 1.27 1.27)) (justify left))
     )
-    (property "Value" "C" (id 1) (at 123.19 90.1699 0)
+    (property "Value" "0.47u" (id 1) (at 123.19 90.1699 0)
       (effects (font (size 1.27 1.27)) (justify left))
     )
@@
     (in_bom yes) (on_board yes) (fields_autoplaced)
     (property "Reference" "C2" (id 0) (at 184.15 138.43 90))
-    (property "Value" "C" (id 1) (at 184.15 140.97 90))
+    (property "Value" "20p" (id 1) (at 184.15 140.97 90))
     (property "Footprint" "Capacitor_SMD:C_0805_2012Metric" (id 2) (at 187.96 145.0848 0)
       (effects (font (size 1.27 1.27)) hide)
@@
       (effects (font (size 1.27 1.27)) (justify left))
     )
-    (property "Value" "C" (id 1) (at 196.85 54.6099 0)
+    (property "Value" "0.1u" (id 1) (at 196.85 54.6099 0)
       (effects (font (size 1.27 1.27)) (justify left))
     )
@@
     (in_bom yes) (on_board yes) (fields_autoplaced)
     (property "Reference" "C8" (id 0) (at 73.66 86.36 90))
-    (property "Value" "C" (id 1) (at 73.66 88.9 90))
+    (property "Value" "20p" (id 1) (at 73.66 88.9 90))
     (property "Footprint" "Capacitor_SMD:C_0805_2012Metric" (id 2) (at 77.47 93.0148 0)
       (effects (font (size 1.27 1.27)) hide)
@@
     (in_bom yes) (on_board yes) (fields_autoplaced)
     (property "Reference" "C4" (id 0) (at 194.31 138.43 90))
-    (property "Value" "C" (id 1) (at 194.31 140.97 90))
+    (property "Value" "20p" (id 1) (at 194.31 140.97 90))
     (property "Footprint" "Capacitor_SMD:C_0805_2012Metric" (id 2) (at 198.12 145.0848 0)
       (effects (font (size 1.27 1.27)) hide)
@@
     )
     (path "/0f9a0d16-15f3-4ae3-8648-0a37cb9b1fcf"
-      (reference "C1") (unit 1) (value "C") (footprint "Capacitor_SMD:C_0805_2012Metric")
+      (reference "C1") (unit 1) (value "0.1u") (footprint "Capacitor_SMD:C_0805_2012Metric")
     )
     (path "/98a8f4e4-ea74-4e33-9e19-1df0a531567e"
-      (reference "C2") (unit 1) (value "C") (footprint "Capacitor_SMD:C_0805_2012Metric")
+      (reference "C2") (unit 1) (value "20p") (footprint "Capacitor_SMD:C_0805_2012Metric")
     )
     (path "/a2084675-d364-42be-93ef-c5b13970963b"
-      (reference "C3") (unit 1) (value "C") (footprint "Capacitor_SMD:C_0805_2012Metric")
+      (reference "C3") (unit 1) (value "0.1u") (footprint "Capacitor_SMD:C_0805_2012Metric")
     )
     (path "/ddbfab92-d93f-4baf-a66b-c6290a34e0d8"
-      (reference "C4") (unit 1) (value "C") (footprint "Capacitor_SMD:C_0805_2012Metric")
+      (reference "C4") (unit 1) (value "20p") (footprint "Capacitor_SMD:C_0805_2012Metric")
     )
     (path "/72984fda-c140-4c53-901b-5af4e1a39aaa"
-      (reference "C5") (unit 1) (value "C") (footprint "Capacitor_SMD:C_0805_2012Metric")
+      (reference "C5") (unit 1) (value "0.1u") (footprint "Capacitor_SMD:C_0805_2012Metric")
     )
     (path "/09f554a4-0999-4ba2-bde9-55a87039208b"
-      (reference "C6") (unit 1) (value "C") (footprint "Capacitor_SMD:C_0805_2012Metric")
+      (reference "C6") (unit 1) (value "0.1u") (footprint "Capacitor_SMD:C_0805_2012Metric")
     )
     (path "/5ad2d851-c8e7-4ae0-8b75-82715d9d6971"
-      (reference "C7") (unit 1) (value "C") (footprint "Capacitor_SMD:C_0805_2012Metric")
+      (reference "C7") (unit 1) (value "20p") (footprint "Capacitor_SMD:C_0805_2012Metric")
     )
     (path "/d2c897d2-0af0-47df-abf7-fe8a795015b3"
-      (reference "C8") (unit 1) (value "C") (footprint "Capacitor_SMD:C_0805_2012Metric")
+      (reference "C8") (unit 1) (value "20p") (footprint "Capacitor_SMD:C_0805_2012Metric")
     )
     (path "/38b24fb7-60a2-443e-8141-810e45c59f35"
-      (reference "C9") (unit 1) (value "C") (footprint "Capacitor_SMD:C_0805_2012Metric")
+      (reference "C9") (unit 1) (value "0.47u") (footprint "Capacitor_SMD:C_0805_2012Metric")
     )
     (path "/84813e82-9923-49a3-853f-badf04a5c21b"
-      (reference "C10") (unit 1) (value "C") (footprint "Capacitor_SMD:C_0805_2012Metric")
+      (reference "C10") (unit 1) (value "0.47u") (footprint "Capacitor_SMD:C_0805_2012Metric")
     )
     (path "/c7254b97-e721-4c70-80a9-e206f127d23f"
@@
     )
     (path "/16b0b8a4-29b7-4458-928b-01b8063192dc"
-      (reference "R1") (unit 1) (value "R") (footprint "Resistor_SMD:R_0805_2012Metric")
+      (reference "R1") (unit 1) (value "4.7K") (footprint "Resistor_SMD:R_0805_2012Metric")
     )
     (path "/248dceca-c537-4498-ac47-c723318e5db2"
-      (reference "R2") (unit 1) (value "R") (footprint "Resistor_SMD:R_0805_2012Metric")
+      (reference "R2") (unit 1) (value "4.7K") (footprint "Resistor_SMD:R_0805_2012Metric")
     )
     (path "/0eedbcbf-cde6-420c-a579-5d2c5bc29faf"
@@
     )
     (path "/44ff6b65-7a5a-4b9c-858a-bee191d7c0d4"
-      (reference "Y1") (unit 1) (value "Crystal") (footprint "Crystal:Crystal_HC49-U_Vertical")
+      (reference "Y1") (unit 1) (value "12Mz") (footprint "Crystal:Crystal_HC49-U_Vertical")
     )
     (path "/835462f5-a49d-41a0-a927-f45c4ed1234c"
-      (reference "Y2") (unit 1) (value "Crystal") (footprint "Crystal:Crystal_HC49-U_Vertical")
-    )
-  )
+      (reference "Y2") (unit 1) (value "12Mz") (footprint "Crystal:Crystal_HC49-U_Vertical")
+    )
+  )
